File: mk-0/KiCAD/TopBoard/Host.kicad_sch (KiCad schematic)
At the start: 8 parts, among them J4 Conn_02x20_Odd_Even, U10 CAT24C256

Commit message: Trace layout complete
Parts:
- added JP23, JP24, JP25, JP26: SolderJumper_2_Bridged, Jumper:SolderJumper-2_P1.3mm_Bridged_RoundedPad1.0x1.5mm, symbol Jumper:SolderJumper_2_Bridged
Connections:
- net at J4.1 (Pin_1): now also JP23.1 (A)
- net at J4.11 (Pin_11): now also JP24.1 (A)
- net at J4.15 (Pin_15): now also JP25.1 (A)
- net at J4.17 (Pin_17): now also JP26.1 (A)
- net MUTE: now reaches J4.36 (Pin_36)
- new net DAC1_M: JP23.2 (B)
- new net DAC1_P: JP24.2 (B)
- new net DAC2_M: JP26.2 (B)
- new net DAC2_P: JP25.2 (B)
- no-connect marks 15 -> 14
