File: mk-0/KiCAD/TopBoard/Mics Mute.kicad_sch (KiCad schematic)
At the start: 59 parts, among them J3 Conn_01x08_MountingPin, Q1 NTR4101P, Q2 FDV301N, SW1 SW_Push, U4 74LVC1G17, U5 74LVC2G74, U6 74LVC125A

Commit message: Trace layout complete
Parts:
- removed JP14, JP15, JP16, JP17, JP18, JP19, JP20, JP21, JP22: SolderJumper_2_Open, Jumper:SolderJumper-2_P1.3mm_Open_RoundedPad1.0x1.5mm, symbol Jumper:SolderJumper_2_Open
- removed R20: 100R, Resistor_SMD:R_0402_1005Metric, symbol Device:R
- added C46, C47, C49: 100nF, Capacitor_SMD:C_0402_1005Metric, symbol Device:C
- added U11: 74LVC125A, Package_SO:SOIC-14_3.9x8.7mm_P1.27mm, symbol 74xx:74LVC125
- R17: value 100R -> 47K; ALTIUM_VALUE 100R -> 47K; MANUFACTURER PART NUMBER RC0402FR-07100RL -> RC0402FR-0747KL; PART NUMBER STD-01-0032 -> STD-01-0096
Connections:
- net +3V3: now also C49.1, U11.14 (VCC)
- net GND: now also R17.2, C46.2, C47.2, C49.2, U11.10, U11.12, U11.13, U11.7 (GND), U11.9
- net MIC_CLK: now also JP2.2 (B), JP4.2 (B), U6.12, U11.2, U11.5; no longer U6.2, U6.5
- net MUTE: now also Q2.1 (G)
- net VDD_MIC: now also MK2.1 (VDD), MK3.1 (VDD), MK5.1 (VDD), MK5.2 (SEL), MK6.1 (VDD), MK6.2 (SEL), C46.1, C47.1; no longer JP12.1 (A), JP8.1 (A)
- net DMIC_IN3_BUF: now reaches R29.2
- net DMIC_IN3_BUF: now also JP13.2 (B), R17.1, R30.2, U6.9
- net DMIC_IN2_BUF: now reaches R28.2
- net DMIC_IN2_BUF: now also JP12.2 (B), R14.1, R33.2, U6.5
- net DMIC_CLK_3: now reaches MK5.3 (CLOCK)
- net DMIC_CLK_3: now also JP4.1 (A), MK3.3 (CLOCK), U11.3
- net DMIC_IN1: now reaches U6.3
- net DMIC_IN1: now also J3.5 (Pin_5), JP8.1 (A)
- net DMIC_IN2: now reaches U6.6
- net DMIC_IN2: now also J3.7 (Pin_7), JP12.1 (A); no longer R17.1
- net DMIC_IN1_BUF: now reaches JP8.2 (B)
- net DMIC_IN1_BUF: now also R10.2, R13.2, R18.1, U6.2; no longer MK2.1 (VDD)
- net DMIC_CLK_2: now reaches MK2.3 (CLOCK)
- net DMIC_CLK_2: now also JP2.1 (A), MK6.3 (CLOCK), U11.6; no longer JP13.1 (A)
- net MIC_CLK_M renamed DMIC_CLK_1
- net DMIC_CLK_1: now also U6.11; no longer JP13.2 (B), R17.2
- removed net MIC_DATA: J3.5 (Pin_5), JP2.2 (B), U6.8
- removed net MIC_DATA2: J3.7 (Pin_7), JP4.2 (B), U6.11
- removed net MIC_DATA2_M: JP4.1 (A), R14.1, U6.12
- removed net MIC_DATA_M: JP2.1 (A), R10.2, R13.2, R18.1, U6.9
- net MUTE_ON renamed MUTE_DATA
- net MUTE_DATA: now also U11.1, U11.4; no longer Q2.1 (G)
- new net DMIC_IN3: JP13.1 (A), U6.8
- no-connect marks 0 -> 2
Other:
- moved on the sheet: C25, C26, C27, C30, C31, C60, C61, C62, D1, FB2, J3, JP1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
