File: mk-0/KiCAD/TopBoard/Signal.kicad_pcb (KiCad board)
At the start: 2 copper layers, 88 x 88 mm, 204 parts, among them J1 Conn_02x10_Odd_Even, J10 AudioJack3, J3 Conn_01x08_MountingPin, J4 Conn_02x20_Odd_Even, J5 USB_C_Receptacle_USB2.0_16P, Q1 NTR4101P, Q2 FDV301N, SW1 SW_Push, SW2 BUTTON 1, SW3 BUTTON 2, SW4 BUTTON 3, U1 W25Q64JVSSIQ, U10 CAT24C256, U16 74AHCT1G125, U2 XU316-1024-QF60B-C24, U3 AP61102, U4 74LVC1G17, U5 74LVC2G74, U6 74LVC125A, U7 TLV320DAC3101, U8 NCP114ASN330, U9 NCP114ASN180, Y1 XRCGB

Commit message: Trace layout complete
Parts:
- removed the C29 at (-37.4, 70.5)
- removed JP14, JP15, JP16, JP17, JP18, JP19, JP20, JP21, JP22: SolderJumper_2_Open, Jumper:SolderJumper-2_P1.3mm_Open_RoundedPad1.0x1.5mm
- removed R20: 100R, Resistor_SMD:R_0402_1005Metric
- added C28: 100nF, Capacitor_SMD:C_0402_1005Metric, F.Cu at (67.5, 102.0)
- added C46: 100nF, Capacitor_SMD:C_0402_1005Metric, F.Cu at (102.0, 72.5)
- added C47: 100nF, Capacitor_SMD:C_0402_1005Metric, F.Cu at (43.6, 51.8)
- added C49: 100nF, Capacitor_SMD:C_0402_1005Metric, F.Cu at (41.7, 77.0)
- added JP23: SolderJumper_2_Bridged, Jumper:SolderJumper-2_P1.3mm_Bridged_RoundedPad1.0x1.5mm, B.Cu at (96.3, 87.5)
- added JP24: SolderJumper_2_Bridged, Jumper:SolderJumper-2_P1.3mm_Bridged_RoundedPad1.0x1.5mm, B.Cu at (93.7, 87.5)
- added JP25: SolderJumper_2_Bridged, Jumper:SolderJumper-2_P1.3mm_Bridged_RoundedPad1.0x1.5mm, B.Cu at (91.2, 87.5)
- added JP26: SolderJumper_2_Bridged, Jumper:SolderJumper-2_P1.3mm_Bridged_RoundedPad1.0x1.5mm, B.Cu at (88.6, 87.5)
- added U11: 74LVC125A, Package_SO:SOIC-14_3.9x8.7mm_P1.27mm, F.Cu at (47.5, 80.2)
- JP12, JP13, JP8: moved to B.Cu
- R17: value 100R -> 47K
- moved R30 154.3 mm to (96.1, 52.7), turned to 30 degrees
- moved C48 143.6 mm to (99.0, 56.2), turned to 30 degrees
- moved R33 139.7 mm to (101.3, 68.0)
- moved JP13 120.0 mm to (59.1, 82.9), turned to 90 degrees
- moved JP8 114.4 mm to (53.7, 77.8), turned to 90 degrees
- moved JP12 114.4 mm to (53.7, 81.6), turned to 90 degrees
- moved C29 114.1 mm to (72.5, 38.0), turned to 90 degrees
- moved R10 112.6 mm to (72.0, 101.3), turned to -90 degrees
- moved R13 107.4 mm to (68.0, 38.7), turned to 90 degrees
- moved R29 101.7 mm to (41.9, 56.1), turned to 150 degrees
- moved C45 82.3 mm to (38.0, 67.5), turned to 180 degrees
- moved R28 80.2 mm to (38.7, 72.0), turned to 180 degrees
- moved R25 49.7 mm to (83.0, 63.0), turned to 180 degrees
- moved R26 48.1 mm to (83.0, 64.0), turned to 0 degrees
- moved R17 29.6 mm to (40.3, 55.1), turned to 150 degrees
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- renumbered C28 to C29
Connections:
- J3 pad 3: /MIC_CLK -> /U_Mics Mute/MIC_CLK
- J3 pad 5: /MIC_DATA -> /U_Mics Mute/DMIC_IN1
- J3 pad 7: /MIC_DATA2 -> /U_Mics Mute/DMIC_IN2
- J4 pad 36: unconnected-(J4-Pin_36-Pad36) -> /U_Mics Mute/MUTE_PWR
- JP1 pad 1: /MIC_CLK -> /U_Mics Mute/MIC_CLK
- JP1 pad 2: /U_Mics Mute/MIC_CLK_M -> /U_Mics Mute/DMIC_CLK_1
- JP12 pad 1: VDD_MIC -> /U_Mics Mute/DMIC_IN2
- JP12 pad 2: Net-(JP12-B) -> /U_Mics Mute/DMIC_IN2_BUF
- JP13 pad 1: Net-(JP13-A) -> /U_Mics Mute/DMIC_IN3
- JP13 pad 2: /U_Mics Mute/MIC_CLK_M -> /U_Mics Mute/DMIC_IN3_BUF
- JP2 pad 1: /U_Mics Mute/MIC_DATA_M -> /U_Mics Mute/DMIC_CLK_2
- JP2 pad 2: /MIC_DATA -> /U_Mics Mute/MIC_CLK
- JP4 pad 1: /U_Mics Mute/MIC_DATA2_M -> /U_Mics Mute/DMIC_CLK_3
- JP4 pad 2: /MIC_DATA2 -> /U_Mics Mute/MIC_CLK
- JP8 pad 1: VDD_MIC -> /U_Mics Mute/DMIC_IN1
- JP8 pad 2: Net-(JP8-B) -> /U_Mics Mute/DMIC_IN1_BUF
- MK1 pad 3: /U_Mics Mute/MIC_CLK_M -> /U_Mics Mute/DMIC_CLK_1
- MK2 pad 1: Net-(JP8-B) -> VDD_MIC
- MK2 pad 3: Net-(JP13-A) -> /U_Mics Mute/DMIC_CLK_2
- MK3 pad 1: Net-(JP17-B) -> VDD_MIC
- MK3 pad 3: Net-(JP19-A) -> /U_Mics Mute/DMIC_CLK_3
- MK4 pad 3: /U_Mics Mute/MIC_CLK_M -> /U_Mics Mute/DMIC_CLK_1
- MK5 pad 1: Net-(JP18-B) -> VDD_MIC
- MK5 pad 2: Net-(JP18-B) -> VDD_MIC
- MK5 pad 3: Net-(JP21-A) -> /U_Mics Mute/DMIC_CLK_3
- MK6 pad 1: Net-(JP12-B) -> VDD_MIC
- MK6 pad 2: Net-(JP12-B) -> VDD_MIC
- MK6 pad 3: Net-(JP15-A) -> /U_Mics Mute/DMIC_CLK_2
- Q2 pad 1: /U_Mics Mute/MUTE_ON -> /U_Mics Mute/MUTE_PWR
- R10 pad 2: /U_Mics Mute/MIC_DATA_M -> /U_Mics Mute/DMIC_IN1_BUF
- R12 pad 2: /U_Mics Mute/MUTE_ON -> /U_Mics Mute/MUTE_DATA
- R13 pad 2: /U_Mics Mute/MIC_DATA_M -> /U_Mics Mute/DMIC_IN1_BUF
- R14 pad 1: /U_Mics Mute/MIC_DATA2_M -> /U_Mics Mute/DMIC_IN2_BUF
- R17 pad 1: Net-(R17-Pad1) -> /U_Mics Mute/DMIC_IN3_BUF
- R17 pad 2: /U_Mics Mute/MIC_CLK_M -> GND
- R18 pad 1: /U_Mics Mute/MIC_DATA_M -> /U_Mics Mute/DMIC_IN1_BUF
- R28 pad 2: Net-(JP14-A) -> /U_Mics Mute/DMIC_IN2_BUF
- R29 pad 2: Net-(JP20-A) -> /U_Mics Mute/DMIC_IN3_BUF
- R30 pad 2: Net-(JP22-A) -> /U_Mics Mute/DMIC_IN3_BUF
- R33 pad 2: Net-(JP16-A) -> /U_Mics Mute/DMIC_IN2_BUF
- R44 pad 2: /MIC_CLK -> /U_Mics Mute/MIC_CLK
- R48 pad 2: /U_Mics Mute/MUTE_ON -> /U_Mics Mute/MUTE_DATA
- U2 pad 11: /MIC_DATA2 -> /U_Mics Mute/DMIC_IN2
- U2 pad 32: /MIC_DATA -> /U_Mics Mute/DMIC_IN1
- U2 pad 46: /MUTE -> /U_Mics Mute/MUTE_PWR
- U5 pad 3: /U_Mics Mute/MUTE_ON -> /U_Mics Mute/MUTE_DATA
- U5 pad 5: /MUTE -> /U_Mics Mute/MUTE_PWR
- U6 pad 1: /U_Mics Mute/MUTE_ON -> /U_Mics Mute/MUTE_DATA
- U6 pad 10: /U_Mics Mute/MUTE_ON -> /U_Mics Mute/MUTE_DATA
- U6 pad 11: /MIC_DATA2 -> /U_Mics Mute/DMIC_CLK_1
- U6 pad 12: /U_Mics Mute/MIC_DATA2_M -> /U_Mics Mute/MIC_CLK
- U6 pad 13: /U_Mics Mute/MUTE_ON -> /U_Mics Mute/MUTE_DATA
- U6 pad 2: /MIC_CLK -> /U_Mics Mute/DMIC_IN1_BUF
- U6 pad 3: Net-(R20-Pad1) -> /U_Mics Mute/DMIC_IN1
- U6 pad 4: /U_Mics Mute/MUTE_ON -> /U_Mics Mute/MUTE_DATA
- U6 pad 5: /MIC_CLK -> /U_Mics Mute/DMIC_IN2_BUF
- U6 pad 6: Net-(R17-Pad1) -> /U_Mics Mute/DMIC_IN2
- U6 pad 8: /MIC_DATA -> /U_Mics Mute/DMIC_IN3
- U6 pad 9: /U_Mics Mute/MIC_DATA_M -> /U_Mics Mute/DMIC_IN3_BUF
Routing:
- net VDD_MIC: track 6.20 -> 204.6 mm, vias 1 -> 11
- net /U_Mics Mute/DMIC_CLK_1: track 0.00 -> 157.5 mm, vias 0 -> 5
- net /U_Mics Mute/DMIC_IN1_BUF: track 0.00 -> 151.6 mm, vias 0 -> 6
- net /U_Mics Mute/DMIC_CLK_2: track 0.00 -> 127.5 mm, vias 0 -> 9
- net /U_Mics Mute/DMIC_IN2_BUF: track 0.00 -> 123.3 mm, vias 0 -> 7
- net /U_Mics Mute/DMIC_IN3_BUF: track 0.00 -> 119.8 mm, vias 0 -> 7
- net /U_Mics Mute/DMIC_CLK_3: track 0.00 -> 116.9 mm, vias 0 -> 7
- net GND: track 116.0 -> 190.5 mm, vias 48 -> 70
- net /MIC_DATA2: track 74.4 -> 0.00 mm, vias 4 -> 0
- net /U_Mics Mute/DMIC_IN2: track 0.00 -> 68.2 mm, vias 0 -> 5
- net /U_Mics Mute/MUTE_PWR: track 0.00 -> 61.2 mm, vias 0 -> 5
- net /U_Mics Mute/MUTE_DATA: track 0.00 -> 52.9 mm, vias 0 -> 4
- net /MIC_DATA: track 51.5 -> 0.00 mm, vias 5 -> 0
- net /U_Mics Mute/MIC_CLK: track 0.00 -> 49.6 mm, vias 0 -> 4
- net /U_Mics Mute/DMIC_IN1: track 0.00 -> 44.9 mm, vias 0 -> 3
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Other:
- board text added: "3V3|1V8|5V"
- board text added: "CUR|0V9"
