File: mk-0/KiCAD/TopBoard/Signal.kicad_sch (KiCad schematic)
At the start: 40 parts, among them SW2 BUTTON 1, SW3 BUTTON 2, SW4 BUTTON 3, U16 74AHCT1G125

Commit message: Trace layout complete
Other:
- sheet U_Host ports: added DAC1_M, DAC1_P, DAC2_M, DAC2_P; removed none
- sheet U_Mics Mute ports: added DMIC_IN1, DMIC_IN2, DMIC_IN3; removed MIC_DATA, MIC_DATA2
- sheet U_XMOS ports: added MIC_DATA3; removed none
Changed lines of the file:
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@@
 	)
 	(junction
+		(at 58.42 138.43)
+		(diameter 0)
+		(color 0 0 0 0)
+	)
+	(junction
 		(at 91.44 58.42)
 		(diameter 0)
@@
 	(wire
 		(pts
+			(xy 58.42 139.7) (xy 58.42 138.43)
+		)
+		(stroke
+			(width 0)
+			(type default)
+		)
+	)
+	(wire
+		(pts
 			(xy 104.14 38.1) (xy 104.14 71.12)
 		)
@@
 	(wire
 		(pts
-			(xy 58.42 127) (xy 195.58 127)
+			(xy 58.42 138.43) (xy 195.58 138.43)
 		)
 		(stroke
@@
 	(wire
 		(pts
+			(xy 175.26 63.5) (xy 203.2 63.5)
+		)
+		(stroke
+			(width 0)
+			(type default)
+		)
+	)
+	(wire
+		(pts
 			(xy 88.9 55.88) (xy 137.16 55.88)
 		)
@@
 	(wire
 		(pts
-			(xy 195.58 66.04) (xy 195.58 127)
+			(xy 195.58 66.04) (xy 195.58 138.43)
 		)
 		(stroke
@@
 		)
 	)
-	(label "MIC_DATA2"
-		(at 177.8 60.96 0)
-		(fields_autoplaced yes)
-		(effects
-			(font
-				(size 1.27 1.27)
-			)
-			(justify left bottom)
-		)
-	)
-	(label "MIC_DATA"
-		(at 177.8 58.42 0)
-		(fields_autoplaced yes)
-		(effects
-			(font
-				(size 1.27 1.27)
-			)
-			(justify left bottom)
-		)
-	)
 	(label "SCL"
 		(at 114.3 55.88 0)
@@
 		)
 	)
-	(label "MIC_CLK"
-		(at 177.8 55.88 0)
-		(fields_autoplaced yes)
-		(effects
-			(font
-				(size 1.27 1.27)
-			)
-			(justify left bottom)
-		)
-	)
 	(label "XVF_RST_N"
 		(at 113.03 121.92 0)
@@
 		)
 	)
-	(label "MUTE"
-		(at 177.8 66.04 0)
-		(fields_autoplaced yes)
-		(effects
-			(font
-				(size 1.27 1.27)
-			)
-			(justify left bottom)
-		)
-	)
 	(symbol
 		(lib_id "power:+5V")
@@
 			)
 		)
+		(pin "MIC_DATA3" input
+			(at 175.26 63.5 0)
+			(effects
+				(font
+					(size 1.27 1.27)
+				)
+				(justify right)
+			)
+		)
 		(instances
 			(project "Signal"
@@
 	(sheet
 		(at 20.32 45.72)
-		(size 38.1 88.9)
+		(size 38.1 93.98)
 		(fields_autoplaced yes)
 		(stroke
@@
 		)
 		(property "Sheetfile" "Host.kicad_sch"
-			(at 20.32 135.2046 0)
+			(at 20.32 140.2846 0)
 			(effects
 				(font
@@
 		)
 		(pin "MUTE" input
-			(at 58.42 127 0)
+			(at 58.42 138.43 0)
 			(effects
 				(font
@@
 			)
 		)
+		(pin "DAC1_M" input
+			(at 58.42 127 0)
+			(effects
+				(font
+					(size 1.27 1.27)
+				)
+				(justify right)
+			)
+		)
+		(pin "DAC1_P" input
+			(at 58.42 129.54 0)
+			(effects
+				(font
+					(size 1.27 1.27)
+				)
+				(justify right)
+			)
+		)
+		(pin "DAC2_P" input
+			(at 58.42 132.08 0)
+			(effects
+				(font
+					(size 1.27 1.27)
+				)
+				(justify right)
+			)
+		)
+		(pin "DAC2_M" input
+			(at 58.42 134.62 0)
+			(effects
+				(font
+					(size 1.27 1.27)
+				)
+				(justify right)
+			)
+		)
 		(instances
 			(project "Signal"
@@
 			)
 		)
-		(pin "MIC_DATA" output
-			(at 203.2 58.42 180)
+		(pin "MUTE" output
+			(at 203.2 66.04 180)
 			(effects
 				(font
@@
 			)
 		)
-		(pin "MUTE" output
-			(at 203.2 66.04 180)
+		(pin "DMIC_IN3" output
+			(at 203.2 63.5 180)
 			(effects
 				(font
@@
 			)
 		)
-		(pin "MIC_DATA2" output
+		(pin "DMIC_IN2" output
 			(at 203.2 60.96 180)
 			(effects
 				(font
+					(size 1.27 1.27)
+				)
+				(justify left)
+			)
+		)
+		(pin "DMIC_IN1" output
+			(at 203.2 58.42 180)
+			(effects
+				(font
