File: mk-0/KiCAD/TopBoard/XMOS.kicad_sch (KiCad schematic)
At the start: 56 parts, among them J1 Conn_02x10_Odd_Even, J5 USB_C_Receptacle_USB2.0_16P, J6 Conn_02x13_Odd_Even, J8 Conn_02x04_Odd_Even, U1 W25Q64JVSSIQ, U2 XU316-1024-QF60B-C24, Y1 XRCGB

Commit message: Trace layout complete
Changed lines of the file:
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@@
+		)
+	)
+	(hierarchical_label "MIC_DATA3"
+		(shape input)
+		(at 294.64 127 0)
+		(fields_autoplaced yes)
+		(effects
+			(font
+				(size 1.27 1.27)
+			)
+			(justify left)
 		)
 	)
